Commit message: fixed collisions, setting resource paths through launch files

File: urdf/bcr_bot.xacro (robot description, xacro)
@@ -18,5 +18,5 @@
     <xacro:property name="traction_wheel_radius" value="0.1"/>
     <xacro:property name="traction_wheel_width" value="0.05"/>
-    <xacro:property name="traction_track_width" value="0.8"/>
+    <xacro:property name="traction_track_width" value="0.6"/>
     <xacro:property name="two_d_lidar_update_rate" value="30"/>
     <xacro:property name="two_d_lidar_sample_size" value="361"/>

File: urdf/macros.xacro (robot description, xacro)
@@ -44,4 +44,5 @@
                     <cylinder length="${traction_wheel_width}" radius="${traction_wheel_radius}"/>
                 </geometry>
+                <self_collide>false</self_collide>
             </collision>
             <inertial>

Commit message: Update robot base frame to base_footprint

File: urdf/bcr_bot.xacro (robot description, xacro)
@@ -41,4 +41,11 @@
     <xacro:include filename="$(find bcr_bot)/urdf/macros.xacro"/>
     <xacro:include filename="$(find bcr_bot)/urdf/gazebo.xacro"/>
+    <!-- ............................. BASE FOOTPRINT ................................ -->
+    <link name="base_footprint"/>
+    <joint name="base_joint" type="fixed">
+      <parent link="base_footprint"/>
+      <child link="base_link"/>
+      <origin xyz="0.0 0.0 0.217" rpy="0 0 0"/>
+    </joint>
     <!-- ................................ BASE LINK .................................. -->
     <link name="base_link"/>

File: urdf/gazebo.xacro (robot description, xacro)
@@ -14,5 +14,5 @@
             <wheelSeparation>${traction_track_width+traction_wheel_width-0.01}</wheelSeparation>
             <wheelDiameter>${2*traction_wheel_radius+0.01}</wheelDiameter>
-            <robotBaseFrame>base_link</robotBaseFrame>
+            <robotBaseFrame>base_footprint</robotBaseFrame>
             <wheelTorque>${traction_max_wheel_torque}</wheelTorque>
             <commandTopic>cmd_vel</commandTopic>

Commit message: Update base_joint origin in bcr_bot.xacro

File: urdf/bcr_bot.xacro (robot description, xacro)
@@ -46,5 +46,5 @@
       <parent link="base_footprint"/>
       <child link="base_link"/>
-      <origin xyz="0.0 0.0 0.217" rpy="0 0 0"/>
+      <origin xyz="0.0 0.0 ${chassis_height/2+2*trolley_wheel_radius+eps}" rpy="0 0 0"/>
     </joint>
     <!-- ................................ BASE LINK .................................. -->
